File: farewell.kicad_pcb (KiCad board)
At the start: 2 copper layers, 215 x 72 mm, 44 parts, among them SW1 SW_Push, U1 0

Commit message: V2 fixes + WS2812 holes in pcb
Parts:
- removed the REF** at (17.0, 106.0)
- removed the REF** at (17.0, 44.0)
- removed the REF** at (79.0, 44.0)
- removed the REF** at (84.7, 93.7)
- removed the REF** at (84.7, 49.4)
- removed the REF** at (154.8, 50.4)
- removed the REF** at (154.8, 94.8)
- removed the REF** at (79.0, 106.0)
- added REF**: breakaway-mousebites, random-kb-part:breakaway-mousebites, F.Cu at (112.5, 111.0)
- added REF**: breakaway-mousebites, random-kb-part:breakaway-mousebites, F.Cu at (112.7, 60.5)
- added REF**: breakaway-mousebites, random-kb-part:breakaway-mousebites, F.Cu at (115.3, 60.5)
- added REF**: breakaway-mousebites, random-kb-part:breakaway-mousebites, F.Cu at (115.3, 111.0)
- added REF**: MountingHole_3.2mm_M3_Pad, Mounting:MountingHole_3.2mm_M3_Pad, F.Cu at (36.5, 48.5)
- added REF**: MountingHole_3.2mm_M3_Pad, Mounting:MountingHole_3.2mm_M3_Pad, F.Cu at (108.5, 124.5)
- added REF**: MountingHole_3.2mm_M3_Pad, Mounting:MountingHole_3.2mm_M3_Pad, F.Cu at (108.5, 48.5)
- added REF**: MountingHole_3.2mm_M3_Pad, Mounting:MountingHole_3.2mm_M3_Pad, F.Cu at (36.5, 124.5)
- SW1: moved to B.Cu
- U1: moved to F.Cu
- moved REF** 107.6 mm to (267.5, 48.5)
- moved REF** 105.2 mm to (191.3, 112.5)
- moved REF** 104.5 mm to (191.5, 62.0)
- moved REF** 49.1 mm to (267.5, 124.5)
- moved RE2 47.7 mm to (173.5, 72.0), turned to 90 degrees
- moved MX3 42.8 mm to (176.0, 112.0)
- moved D9 42.4 mm to (176.0, 121.5)
- moved SW1 42.0 mm to (179.5, 52.5)
- moved REF** 41.0 mm to (188.7, 112.5)
- moved GND_RST1 40.8 mm to (172.5, 48.5)
- moved MX6 40.6 mm to (176.0, 88.0)
- moved D8 40.2 mm to (176.0, 97.5)
- moved REF** 40.0 mm to (195.5, 124.5)
- moved D7 39.5 mm to (176.5, 76.0)
- moved EXT1 39.4 mm to (146.0, 51.0)
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Connections:
- MX4 pad 1: Net-(MX4-Pad1) -> COL0
- MX5 pad 1: Net-(MX5-Pad1) -> COL1
- MX6 pad 1: Net-(MX6-Pad1) -> COL2
- MX7 pad 1: Net-(MX7-Pad1) -> COL0
- MX8 pad 1: Net-(MX8-Pad1) -> COL1
- MX9 pad 1: Net-(MX9-Pad1) -> COL2
- U1 pad 10: COL2 -> Net-(U1-Pad10)
- U1 pad 11: COL1 -> E1A
- U1 pad 12: COL0 -> E1B
- U1 pad 13: ROW0 -> ROW2
- U1 pad 15: ROW2 -> ROW0
- U1 pad 16: Net-(U1-Pad16) -> E2B
- U1 pad 18: E2B -> COL0
- U1 pad 19: E1A -> COL1
- U1 pad 20: E1B -> COL2
- U1 pad 23: E_G1 -> E_G2
- U1 pad 3: E_G2 -> Net-(U1-Pad3)
- U1 pad 4: Net-(U1-Pad4) -> E_G1
Routing:
- net (no net): track 195.4 -> 1.33 mm
- net Net-(EXT1-Pad1): track 2.68 -> 49.7 mm
- net VCC: track 42.9 -> 0.00 mm, vias 2 -> 0
- net Net-(SCL1-Pad1): track 3.00 -> 39.6 mm
- net ROW0: track 74.9 -> 105.9 mm
- net E_G1: track 7.15 -> 33.8 mm
- net Net-(SDA1-Pad1): track 3.20 -> 27.4 mm
- net ROW1: track 58.9 -> 80.1 mm
- net ADC2: track 16.1 -> 0.00 mm
- net COL2: track 82.2 -> 96.8 mm
- net ADC1: track 10.9 -> 0.00 mm
- net Net-(SW1-Pad1): track 63.6 -> 52.9 mm, vias 2 -> 0
- net ROW2: track 50.7 -> 59.9 mm
- net E1B: track 3.42 -> 12.3 mm
- net E2B: track 71.0 -> 79.0 mm
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Other:
- board size 215 x 72 mm -> 239 x 84 mm
