File: farewell.sch (KiCad schematic (older format))
At the start: 27 parts, among them SW1 SW_Push, U1 0

Commit message: [WIP] Added RGB plate
Parts:
- added RGB1, RGB2, RGB3, RGB4, RGB5, RGB6, RGB7, RGB8, RGB9: WS2812B, LED_SMD:LED_WS2812B_PLCC4_5.0x5.0mm_P3.2mm, symbol LED:WS2812B
- added RGB_DI1, RGB_DI_MCU1, RGB_GND1, RGB_GND_MCU1, RGB_VCC1, RGB_VCC_MCU1: Conn_01x01, keyboard_parts:PIN_1, symbol Connector_Generic:Conn_01x01
Connections:
- net COL0: now also MX4.1, MX7.1, U1.18 (F6); no longer U1.12 (B5)
- net COL1: now also MX5.1, MX8.1, U1.19 (F5); no longer U1.11 (B4)
- net COL2: now also MX6.1, MX9.1, U1.20 (F4); no longer U1.10 (E6)
- net E1A: now also U1.11 (B4); no longer U1.19 (F5)
- net E1B: now also U1.12 (B5); no longer U1.20 (F4)
- net E2B: now also U1.16 (B1); no longer U1.18 (F6)
- net E_G1: now also U1.4 (GND); no longer U1.23 (GND)
- net E_G2: now also U1.23 (GND); no longer U1.3 (GND)
- net ROW0: now also U1.15 (B3); no longer U1.13 (B6)
- net ROW2: now also U1.13 (B6); no longer U1.15 (B3)
- net VCC: now also RGB_VCC_MCU1.1 (Pin_1)
- new net: RGB_DI_MCU1.1 (Pin_1), U1.10 (E6)
- new net: RGB_GND_MCU1.1 (Pin_1), U1.3 (GND)
- new net: RGB1.1 (VDD), RGB2.1 (VDD), RGB3.1 (VDD), RGB4.1 (VDD), RGB5.1 (VDD), RGB6.1 (VDD), RGB7.1 (VDD), RGB8.1 (VDD), RGB9.1 (VDD), RGB_VCC1.1 (Pin_1)
- new net: RGB1.2 (DOUT), RGB2.4 (DIN)
- new net: RGB1.3 (VSS), RGB2.3 (VSS), RGB3.3 (VSS), RGB4.3 (VSS), RGB5.3 (VSS), RGB6.3 (VSS), RGB7.3 (VSS), RGB8.3 (VSS), RGB9.3 (VSS), RGB_GND1.1 (Pin_1)
- new net: RGB1.4 (DIN), RGB_DI1.1 (Pin_1)
- new net: RGB2.2 (DOUT), RGB3.4 (DIN)
- new net: RGB3.2 (DOUT), RGB4.4 (DIN)
- new net: RGB6.2 (DOUT), RGB7.4 (DIN)
- new net: RGB5.2 (DOUT), RGB6.4 (DIN)
- new net: RGB8.2 (DOUT), RGB9.4 (DIN)
- new net: RGB7.2 (DOUT), RGB8.4 (DIN)
- new net: RGB4.2 (DOUT), RGB5.4 (DIN)
Other:
- moved on the sheet: GND_RST1
