File: farewell.sch (KiCad schematic (older format))
At the start: 48 parts, among them J1 Conn_01x08, J2 Conn_01x08, J3 Conn_01x06, J4 Conn_01x06, SW1 SW_Push, U1 0

Commit message: Complete pcb
Parts:
- removed EXT1: Conn_01x01, keyboard_parts:PIN_1, symbol Connector_Generic:Conn_01x01
- removed J1, J2: Conn_01x08, farewell_pcb:keebio_Header-8-Pin-ZigZag, symbol Connector_Generic:Conn_01x08
- removed J3, J4: Conn_01x06, farewell_pcb:keebio_Header-6-Pin-ZigZag, symbol Connector_Generic:Conn_01x06
- removed SW1: SW_Push, random-kb-part:PushButton_6x6mm_TH_Pretty, symbol Switch:SW_Push
- MX1, MX2, MX3, MX4, MX5, MX6, MX7, MX8, MX9: footprint keebio:MX-Alps-Choc-1U-NoLED -> farewell_pcb:MX-Alps-Choc-1U-NoLED-noprongs
Connections:
- net ADC1_MCU is gone; now on net ADC1_SW: U1.10 (E6)
- net ADC2_MCU is gone; now on net ADC2_SW: U1.11 (B4)
- net COL0_MCU is gone; now on net COL0_SW: U1.8 (C6)
- net COL1_MCU is gone; now on net COL1_SW: U1.7 (D4)
- net COL2_MCU is gone; now on net COL2_SW: U1.19 (F5)
- net E1A_MCU is gone; now on net E1A_SW: U1.12 (B5)
- net E1B_MCU is gone; now on net E1B_SW: U1.13 (B6)
- net E2A_MCU is gone; now on net E2A_SW: U1.18 (F6)
- net E2B_MCU is gone; now on net E2B_SW: U1.17 (F7)
- net GND_SW is gone; now on net GND: JOY1.H3 (H-), JOY1.V3 (V-), RE1.C, RE2.C
- net ROW0_MCU is gone; now on net ROW0_SW: U1.14 (B2)
- net ROW1_MCU is gone; now on net ROW1_SW: U1.15 (B3)
- net ROW2_MCU is gone; now on net ROW2_SW: U1.16 (B1)
- net VCC_SW is gone; now on net VCC: JOY1.H1 (H+), JOY1.V1 (V+)
- net GND: now also C1.2
- net RGB_VCC: now also U1.24 (RAW)
- net VCC_MCU renamed VCC
Other:
- moved on the sheet: C1
